File: Schematic/Drum_Machine_V01/Drum_Machine.sch (EAGLE design)
At the start: 315 parts, among them CN1 USBA_FEMALE, CN4 MicroUSB, IC1 74595N, IC2 74595N, IC3 74595N, IC4 74595N, IC9 74LS165D, J1 USB-A-SMD, J2 M10SILK_FEMALE_PTH, Q00 BC857CSMD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

Commit message: Updated connections
Parts:
- added J5, J6: 22-23-2031, con-molex:22-23-2031
Connections:
- removed net DATA/MOSI: IC1.SER
- new net AUDIO_HPL: J6-2.S
- new net AUDIO_HPR: J6-3.S
- new net AUDIO_INL: J5-2.S
- new net AUDIO_INR: J5-3.S
- new net D3: P2.6
- new net D4: P2.8
- new net D5: P2.10
- new net D6: P2.18
- new net D7: P2.20
- new net DATA_IN: P2.27
- new net DATA_OUT: IC1.SER, P2.25
- new net LOAD: P2.22
- new net MOTOR_DIR: P2.2
- new net MOTOR_EN: P2.4
- new net MOTOR_PWM: P2.1
- net CLOCK: now also P2.29
- net GND: now also IC3.GND, IC4.GND, J5-1.S, J6-1.S
- net LATCH: now also P2.24
- net N$124: no longer IC3.GND, IC4.GND
Other:
- note added: "Analog input headder"
- note added: "Audio connections"
- note added: "Audio in"
- note added: "Audio out"
- note added: "Headders viewed from bottom of Pocket Beagle"
- note added: "SPI1"
- moved on the sheet: D40, J1, J2, P1, P2, R101, R102
