File: Schematic/Drum_Machine_V01/Drum_Machine.sch (EAGLE design)
At the start: 317 parts, among them CN1 USBA_FEMALE, CN4 MicroUSB, IC1 74595N, IC2 74595N, IC3 74595N, IC4 74595N, IC9 74LS165D, J1 USB-A-SMD, J2 M10SILK_FEMALE_PTH, J5 22-23-2031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

Commit message: Added enclosure and 3D files
Parts:
- added JP1: (no value), adafruit:PINHD-1X8-3.5MM
- added JP2, JP3: (no value), pinhead:PINHD-1X5/90
- added JP4: (no value), pinhead:PINHD-2X5/90
- added JP5, JP6: (no value), pinhead:PINHD-1X8/90
Other:
- note added: "Board Interconnects"
Changed lines of the file:
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@@
 <part name="AGND3" library="supply1" deviceset="AGND" device=""/>
 <part name="J6" library="con-molex" deviceset="22-23-2031" device=""/>
+<part name="FRAME2" library="frames" library_urn="urn:adsk.eagle:library:229" deviceset="LETTER_L" device=""/>
+<part name="JP1" library="adafruit" deviceset="PINHD-1X8" device="-3.5MM"/>
+<part name="JP2" library="pinhead" library_urn="urn:adsk.eagle:library:325" deviceset="PINHD-1X5" device="/90" package3d_urn="urn:adsk.eagle:package:22467/2"/>
+<part name="JP3" library="pinhead" library_urn="urn:adsk.eagle:library:325" deviceset="PINHD-1X5" device="/90" package3d_urn="urn:adsk.eagle:package:22467/2"/>
+<part name="JP4" library="pinhead" library_urn="urn:adsk.eagle:library:325" deviceset="PINHD-2X5" device="/90" package3d_urn="urn:adsk.eagle:package:22471/2"/>
+<part name="JP5" library="pinhead" library_urn="urn:adsk.eagle:library:325" deviceset="PINHD-1X8" device="/90" package3d_urn="urn:adsk.eagle:package:22413/2"/>
+<part name="JP6" library="pinhead" library_urn="urn:adsk.eagle:library:325" deviceset="PINHD-1X8" device="/90" package3d_urn="urn:adsk.eagle:package:22413/2"/>
 </parts>
 <sheets>
@@
 </nets>
 </sheet>
+<sheet>
+<description>Board Interconnects</description>
+<plain>
+<text x="152.4" y="27.94" size="2.54" layer="94">Board Interconnects</text>
+<wire x1="114.3" y1="172.72" x2="114.3" y2="116.84" width="0.1524" layer="98"/>
+<wire x1="114.3" y1="116.84" x2="223.52" y2="116.84" width="0.1524" layer="98"/>
+<wire x1="223.52" y1="116.84" x2="223.52" y2="172.72" width="0.1524" layer="98"/>
+<wire x1="223.52" y1="172.72" x2="114.3" y2="172.72" width="0.1524" layer="98"/>
+</plain>
+<instances>
+<instance part="FRAME2" gate="G$1" x="0" y="0"/>
+<instance part="FRAME2" gate="G$2" x="147.32" y="0"/>
+<instance part="JP1" gate="G$1" x="66.04" y="73.66" rot="R270"/>
+<instance part="JP2" gate="A" x="139.7" y="162.56" rot="R270"/>
+<instance part="JP3" gate="A" x="124.46" y="157.48"/>
+<instance part="JP4" gate="A" x="167.64" y="78.74" rot="R270"/>
+<instance part="JP5" gate="A" x="124.46" y="129.54"/>
+<instance part="JP6" gate="A" x="205.74" y="162.56" rot="R270"/>
+</instances>
+<busses>
+</busses>
+<nets>
+</nets>
+</sheet>
