File: Schematic/Drum_Machine_V01/Drum_Machine.brd (EAGLE design)
At the start: 400 x 190 mm, 315 parts, among them CN1 USBA_FEMALE, CN4 MicroUSB, IC1 74595N, IC2 74595N, IC3 74595N, IC4 74595N, IC9 74LS165D, J1 USB-A-SMD, J2 M10SILK_FEMALE_PTH, Q00 BC857CSMD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

Commit message: Updated connections
Parts:
- added J5, J6: 22-23-2031, con-molex:22-23-2031
Connections:
- removed net DATA/MOSI: IC1.14
- new net AUDIO_HPL: J6.2
- new net AUDIO_HPR: J6.3
- new net AUDIO_INL: J5.2
- new net AUDIO_INR: J5.3
- new net D3: P2.6
- new net D4: P2.8
- new net D5: P2.10
- new net D6: P2.18
- new net D7: P2.20
- new net DATA_IN: P2.27
- new net DATA_OUT: IC1.14, P2.25
- new net LOAD: P2.22
- new net MOTOR_DIR: P2.2
- new net MOTOR_EN: P2.4
- new net MOTOR_PWM: P2.1
- net CLOCK: now also P2.29
- net GND: now also IC3.8, IC4.8, J5.1, J6.1
- net LATCH: now also P2.24
- net N$124: no longer IC3.8, IC4.8
Changed lines of the file:
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@@
 <element name="R11" library="adafruit" package="0204/5" value="" x="-249" y="-593"/>
 <element name="R12" library="adafruit" package="0204/5" value="" x="-249" y="-610"/>
+<element name="J5" library="con-molex" package="22-23-2031" value="22-23-2031" x="-250" y="-672">
+<attribute name="MF" value="MOLEX" x="-250" y="-672" size="1.778" layer="27" display="off"/>
+<attribute name="MPN" value="22-23-2031" x="-250" y="-672" size="1.778" layer="27" display="off"/>
+<attribute name="OC_FARNELL" value="1462950" x="-250" y="-672" size="1.778" layer="27" display="off"/>
+<attribute name="OC_NEWARK" value="30C0862" x="-250" y="-672" size="1.778" layer="27" display="off"/>
+</element>
+<element name="J6" library="con-molex" package="22-23-2031" value="22-23-2031" x="-250" y="-688">
+<attribute name="MF" value="MOLEX" x="-250" y="-688" size="1.778" layer="27" display="off"/>
+<attribute name="MPN" value="22-23-2031" x="-250" y="-688" size="1.778" layer="27" display="off"/>
+<attribute name="OC_FARNELL" value="1462950" x="-250" y="-688" size="1.778" layer="27" display="off"/>
+<attribute name="OC_NEWARK" value="30C0862" x="-250" y="-688" size="1.778" layer="27" display="off"/>
+</element>
 </elements>
 <signals>
@@
 <contactref element="R10" pad="2"/>
 <contactref element="R9" pad="2"/>
+<contactref element="IC4" pad="8"/>
+<contactref element="IC3" pad="8"/>
+<contactref element="J5" pad="1"/>
+<contactref element="J6" pad="1"/>
+<wire x1="616.585" y1="142.875" x2="626.745" y2="135.255" width="0" layer="19" extent="1-1"/>
 <wire x1="610.025" y1="125.005" x2="616.585" y2="142.875" width="0" layer="19" extent="1-1"/>
 <wire x1="609.175" y1="125.005" x2="610.025" y2="125.005" width="0" layer="19" extent="1-1"/>
-<wire x1="647.7" y1="142.875" x2="616.585" y2="142.875" width="0" layer="19" extent="1-1"/>
+<wire x1="647.7" y1="142.875" x2="626.745" y2="135.255" width="0" layer="19" extent="1-1"/>
+<wire x1="657.86" y1="135.255" x2="647.7" y2="142.875" width="0" layer="19" extent="1-1"/>
 <wire x1="530.225" y1="88.7984" x2="609.175" y2="125.005" width="0" layer="19" extent="1-1"/>
 <wire x1="531.495" y1="82.6516" x2="530.225" y2="88.7984" width="0" layer="19" extent="1-1"/>
@@
 <wire x1="-246.46" y1="-559" x2="-210.14" y2="-529.35" width="0" layer="19" extent="1-1"/>
 <wire x1="-246.46" y1="-576" x2="-246.46" y2="-559" width="0" layer="19" extent="1-1"/>
+<wire x1="-252.54" y1="-672" x2="-246.46" y2="-576" width="0" layer="19" extent="1-1"/>
+<wire x1="-252.54" y1="-688" x2="-252.54" y2="-672" width="0" layer="19" extent="1-1"/>
 </signal>
 <signal name="5.0V">
@@
 <contactref element="IC1" pad="8"/>
 <contactref element="IC2" pad="8"/>
-<contactref element="IC3" pad="8"/>
-<contactref element="IC4" pad="8"/>
-<wire x1="657.86" y1="135.255" x2="626.745" y2="135.255" width="0" layer="19" extent="1-1"/>
-<wire x1="267.97" y1="90.805" x2="626.745" y2="135.255" width="0" layer="19" extent="1-1"/>
-<wire x1="38.1" y1="325.12" x2="267.97" y2="90.805" width="0" layer="19" extent="1-1"/>
+<wire x1="267.97" y1="90.805" x2="38.1" y2="325.12" width="0" layer="19" extent="1-1"/>
 </signal>
 <signal name="N$132">
@@
 <contactref element="IC1" pad="11"/>
 <contactref element="IC2" pad="11"/>
-<wire x1="262.89" y1="98.425" x2="33.02" y2="332.74" width="0" layer="19" extent="1-1"/>
-<wire x1="523.875" y1="82.6516" x2="262.89" y2="98.425" width="0" layer="19" extent="1-1"/>
+<contactref element="P2" pad="29"/>
+<wire x1="262.89" y1="98.425" x2="285.115" y2="178.435" width="0" layer="19" extent="1-1"/>
+<wire x1="523.875" y1="82.6516" x2="285.115" y2="178.435" width="0" layer="19" extent="1-1"/>
 <wire x1="621.665" y1="142.875" x2="523.875" y2="82.6516" width="0" layer="19" extent="1-1"/>
 <wire x1="652.78" y1="142.875" x2="621.665" y2="142.875" width="0" layer="19" extent="1-1"/>
+<wire x1="33.02" y1="332.74" x2="285.115" y2="178.435" width="0" layer="19" extent="1-1"/>
 </signal>
 <signal name="LATCH">
@@
 <contactref element="IC1" pad="12"/>
 <contactref element="IC2" pad="12"/>
+<contactref element="P2" pad="24"/>
 <wire x1="650.24" y1="142.875" x2="619.125" y2="142.875" width="0" layer="19" extent="1-1"/>
-<wire x1="260.35" y1="98.425" x2="619.125" y2="142.875" width="0" layer="19" extent="1-1"/>
-<wire x1="30.48" y1="332.74" x2="260.35" y2="98.425" width="0" layer="19" extent="1-1"/>
+<wire x1="277.495" y1="180.975" x2="619.125" y2="142.875" width="0" layer="19" extent="1-1"/>
+<wire x1="260.35" y1="98.425" x2="277.495" y2="180.975" width="0" layer="19" extent="1-1"/>
+<wire x1="30.48" y1="332.74" x2="277.495" y2="180.975" width="0" layer="19" extent="1-1"/>
 </signal>
 <signal name="N$33">
@@
 <wire x1="35" y1="20" x2="251.03" y2="89.535" width="0" layer="19" extent="1-1"/>
 </signal>
-<signal name="DATA/MOSI">
+<signal name="DATA_OUT">
 <contactref element="IC1" pad="14"/>
+<contactref element="P2" pad="25"/>
+<wire x1="25.4" y1="332.74" x2="280.035" y2="178.435" width="0" layer="19" extent="1-1"/>
 </signal>
 <signal name="N$22">
@@
 <wire x1="-246.46" y1="-610" x2="-251.54" y2="-576" width="0" layer="19" extent="1-1"/>
 </signal>
+<signal name="MOTOR_PWM">
+<contactref element="P2" pad="1"/>
+</signal>
+<signal name="MOTOR_EN">
+<contactref element="P2" pad="4"/>
+</signal>
+<signal name="DATA_IN">
+<contactref element="P2" pad="27"/>
+</signal>
+<signal name="LOAD">
+<contactref element="P2" pad="22"/>
+</signal>
+<signal name="D7">
+<contactref element="P2" pad="20"/>
+</signal>
+<signal name="D6">
+<contactref element="P2" pad="18"/>
+</signal>
+<signal name="D5">
+<contactref element="P2" pad="10"/>
+</signal>
+<signal name="D4">
+<contactref element="P2" pad="8"/>
+</signal>
+<signal name="MOTOR_DIR">
+<contactref element="P2" pad="2"/>
+</signal>
+<signal name="D3">
+<contactref element="P2" pad="6"/>
+</signal>
+<signal name="AUDIO_INR">
+<contactref element="J5" pad="3"/>
+</signal>
+<signal name="AUDIO_INL">
+<contactref element="J5" pad="2"/>
+</signal>
+<signal name="AUDIO_HPL">
+<contactref element="J6" pad="2"/>
+</signal>
+<signal name="AUDIO_HPR">
+<contactref element="J6" pad="3"/>
+</signal>
 </signals>

Commit message: Added enclosure and 3D files
Parts:
- added JP1: (no value), adafruit:1X08-3.5MM
- added JP2, JP3: (no value), pinhead:1X05/90
- added JP4: (no value), pinhead:2X05/90
- added JP5, JP6: (no value), pinhead:1X08/90
- moved J5 984.3 mm to (-51.0, 292.0)
- moved J6 984.3 mm to (-51.0, 276.0)
- moved Q24 368.3 mm to (159.8, 525.7)
- moved Q25 368.3 mm to (178.2, 525.7)
- moved Q26 368.3 mm to (196.6, 525.7)
- moved C19 368.3 mm to (190.4, 372.3)
- moved C5 368.3 mm to (737.0, 394.2)
- moved CN1 368.3 mm to (224.1, 371.1)
- moved CN4 368.3 mm to (186.9, 370.1)
- moved D1 368.3 mm to (147.7, 290.4)
- moved D10 368.3 mm to (170.2, 273.9)
- moved D11 368.3 mm to (192.5, 265.7)
- moved D12 368.3 mm to (203.3, 274.2)
- moved D13 368.3 mm to (188.6, 272.6)
- moved D14 368.3 mm to (210.2, 283.1)
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Other:
- board size 400 x 190 mm -> 615 x 622 mm
- board text added: "Button Matrix Board"
- board text added: "LED Driver Board"
